Commit message: Changed ur5-Files to work with MiR - not working yet. Added code in robot_control to make camera work on MiR-Core with python-wrapper

File: coffee_on_table/ur5_Files/ur5.urdf.xacro (robot description, xacro)
@@ -74,5 +74,5 @@
      wrist_2_lower_limit:=${-pi}    wrist_2_upper_limit:=${pi}
      wrist_3_lower_limit:=${-pi}    wrist_3_upper_limit:=${pi}">
-    <link name="${prefix}base_link" >
+    <link name="${prefix}base_link_ur" >
       <visual>
         <geometry>
@@ -93,5 +93,5 @@
     </link>
     <joint name="${prefix}shoulder_pan_joint" type="revolute">
-      <parent link="${prefix}base_link" />
+      <parent link="${prefix}base_link_ur" />
       <child link = "${prefix}shoulder_link" />
       <origin xyz="0.0 0.0 ${shoulder_height}" rpy="0.0 0.0 0.0" />
@@ -309,5 +309,5 @@
     <!-- ROS base_link to UR 'Base' Coordinates transform -->
     <link name="${prefix}base"/>
-    <joint name="${prefix}base_link-base_fixed_joint" type="fixed">
+    <joint name="${prefix}base_link_ur-base_fixed_joint" type="fixed">
       <!-- NOTE: this rotation is only needed as long as base_link itself is
                  not corrected wrt the real robot (ie: rotated over 180
@@ -315,5 +315,5 @@
       -->
       <origin xyz="0 0 0" rpy="0 0 ${-pi}"/>
-      <parent link="${prefix}base_link"/>
+      <parent link="${prefix}base_link_ur"/>
       <child link="${prefix}base"/>
     </joint>
