Commit message: Added urdf-Code to make ur and MiR work together. Currently still bugs when launching simulation. Code for real robots missing.

File: coffee_on_table/urdf/mir_ur5.urdf.xacro (robot description, xacro)
@@ -1,15 +1,30 @@
 <?xml version="1.0"?>
-<robot xmlns:xacro="http://ros.org/wiki/xacro" name="mir_ur5">
+<robot xmlns:xacro="http://ros.org/wiki/xacro" name="ur5">
+  <!-- common stuff -->
+  <xacro:include filename="$(find ur_description)/urdf/common.gazebo.xacro" />
+  <xacro:include filename="$(find mir_description)/urdf/include/common.gazebo.xacro" />
   <!-- include macros for M-10iA and the eef model -->
-  <xacro:include filename="$(find mir_description)/urdf/mir.urdf.xacro"/>
-  <xacro:include filename="$(find ur_description)/urdf/ur5_robot.urdf.xacro" />
-  <!-- create the robot + eef combo itself as a macro -->
+  <!-- MiR100 base -->
+  <xacro:include filename="$(find mir_description)/urdf/include/mir_100_v1.urdf.xacro" />
+  <xacro:mir_100 prefix=""/>
+  <xacro:controller_plugin_gazebo robot_namespace=""/>
+  <!-- ur5 -->
+  <xacro:include filename="$(find ur_description)/urdf/ur5.urdf.xacro" />
+  <xacro:ur5_robot prefix="" joint_limited="false"/>
+  <!-- arm -->
+  <!--<xacro:ur5_robot prefix="" joint_limited="false"/>-->
+  <link name="world" />
+  <joint name="world_joint" type="fixed">
+    <parent link="world" />
+    <child link = "base_link_ur" />
+    <origin xyz="0.0 0.0 0.0" rpy="0.0 0.0 0.0" />
+  </joint>-->
     <!-- attach eef to M-10iA model -->
     <!-- Note: this assumes that the 'my_eef' macro defines a 'base_link'
          link which is the start of it's kinematic chain (if any) -->
     <joint name="compJoint" type="fixed">
-      <origin xyz="0 0 0" rpy="0 0 0" />
+      <origin xyz="0 0 0.5" rpy="0 0 0" />
       <parent link="base_footprint" />
-      <child link="base_link_ur" />
+      <child link="world" />
     </joint>
 </robot>

Commit message: Changed position of UR to MiR. Changed rviz file tf config. Added code in mir_control to subscribe to objPose relative to origin and changed robot_control accordingly. Now the limited UR-model is called

File: coffee_on_table/urdf/mir_ur5.urdf.xacro (robot description, xacro)
@@ -4,5 +4,4 @@
   <xacro:include filename="$(find ur_description)/urdf/common.gazebo.xacro" />
   <xacro:include filename="$(find mir_description)/urdf/include/common.gazebo.xacro" />
-  <!-- include macros for M-10iA and the eef model -->
   <!-- MiR100 base -->
   <xacro:include filename="$(find mir_description)/urdf/include/mir_100_v1.urdf.xacro" />
@@ -11,7 +10,14 @@
   <!-- ur5 -->
   <xacro:include filename="$(find ur_description)/urdf/ur5.urdf.xacro" />
-  <xacro:ur5_robot prefix="" joint_limited="false"/>
-  <!-- arm -->
-  <!--<xacro:ur5_robot prefix="" joint_limited="false"/>-->
+  <!--NOT LIMITED<xacro:ur5_robot prefix="" joint_limited="false"/>-->
+  <xacro:ur5_robot prefix="" joint_limited="true"
+    shoulder_pan_lower_limit="${-pi}" shoulder_pan_upper_limit="${pi}"
+    shoulder_lift_lower_limit="${-pi}" shoulder_lift_upper_limit="${pi}"
+    elbow_joint_lower_limit="${-pi}" elbow_joint_upper_limit="${pi}"
+    wrist_1_lower_limit="${-pi}" wrist_1_upper_limit="${pi}"
+    wrist_2_lower_limit="${-pi}" wrist_2_upper_limit="${pi}"
+    wrist_3_lower_limit="${-pi}" wrist_3_upper_limit="${pi}"
+  />
+  <!-- Connection UR to planning frame world -->
   <link name="world" />
   <joint name="world_joint" type="fixed">
@@ -20,10 +26,8 @@
     <origin xyz="0.0 0.0 0.0" rpy="0.0 0.0 0.0" />
   </joint>-->
-    <!-- attach eef to M-10iA model -->
-    <!-- Note: this assumes that the 'my_eef' macro defines a 'base_link'
-         link which is the start of it's kinematic chain (if any) -->
+  <!-- Connection MiR to world where UR is connected -->
     <joint name="compJoint" type="fixed">
-      <origin xyz="0 0 0.5" rpy="0 0 0" />
-      <parent link="base_footprint" />
+      <origin xyz="0.153 -0.0325 0.892" rpy="0 0 0" /> <!-- 0.892 = 0.352 + 0.54 ; 0.153 = 0.038 + 0,115-->
+      <parent link="base_link" />
       <child link="world" />
     </joint>

Commit message: Changed tf-transforms to fit new eef-pose. Included Box and EEF in Visualisation for collission-detection. Included EEF in ur5-files for eef-point-planning

File: coffee_on_table/urdf/mir_ur5.urdf.xacro (robot description, xacro)
@@ -19,4 +19,6 @@
     wrist_3_lower_limit="${-pi}" wrist_3_upper_limit="${pi}"
   />
+  <!-- Controlbox -->
+  <xacro:include filename="$(find coffee_on_table)/urdf/controlbox.urdf" />
   <!-- Connection UR to planning frame world -->
   <link name="world" />
@@ -25,10 +27,16 @@
     <child link = "base_link_ur" />
     <origin xyz="0.0 0.0 0.0" rpy="0.0 0.0 0.0" />
-  </joint>-->
+  </joint>
   <!-- Connection MiR to world where UR is connected -->
-    <joint name="compJoint" type="fixed">
-      <origin xyz="0.153 -0.0325 0.892" rpy="0 0 0" /> <!-- 0.892 = 0.352 + 0.54 ; 0.153 = 0.038 + 0,115-->
-      <parent link="base_link" />
-      <child link="world" />
-    </joint>
+  <joint name="compJoint" type="fixed">
+    <origin xyz="0.153 -0.0325 0.892" rpy="0 0 0" /> <!-- 0.153 = 0.038 + 0.115; - ; 0.892 = 0.352 + 0.54-->
+    <parent link="base_link" />
+    <child link="world" />
+  </joint>
+  <!-- Connection controlbox to MiR -->
+  <joint name="boxJoint" type="fixed">
+    <origin xyz="0.038 0 0.352" rpy="0 0 0" />
+    <parent link="base_link" />
+    <child link="controlbox" />
+  </joint>
 </robot>

File: universal_robot/ur_description/urdf/ur5.urdf.xacro (robot description, xacro)
@@ -291,4 +291,42 @@
       </collision>
     </link>
+    <!-- Added for planning with gripper as eef -->
+    <joint name="${prefix}gripper_fixed_joint" type="fixed">
+      <parent link="${prefix}wrist_3_link" />
+      <child link = "${prefix}gripper" />
+      <origin xyz="0.0 ${wrist_3_length + 0.144} 0.0" rpy="0.0 0.0 ${pi/2.0}" />
+    </joint>
+    <link name="${prefix}gripper">
+      <collision>
+        <geometry>
+          <box size="0.01 0.01 0.01"/>
+        </geometry>
+        <origin rpy="0 0 0" xyz="-0.01 0 0"/>
+      </collision>
+    </link>
+    <!-- Added for showing eef -->
+    <joint name="${prefix}eef_fixed_joint" type="fixed">
+      <parent link="${prefix}wrist_3_link" />
+      <child link = "${prefix}eef" />
+      <origin xyz="0.0 ${wrist_3_length} 0.0" rpy="${pi/2.0} 0.0 ${pi/2.0}" />
+    </joint>
+    <link name="${prefix}eef">
+      <visual>
+        <geometry>
+          <mesh filename="package://ur_description/meshes/EEF.STL" scale="0.001 0.001 0.001"/>
+        </geometry>
+        <material name="LightGrey">
+          <color rgba="0.7 0.7 0.7 1.0"/>
+        </material>
+      </visual>
+      <collision>
+        <geometry>
+          <mesh filename="package://ur_description/meshes/EEF.STL" scale="0.001 0.001 0.001"/>
+        </geometry>
+      </collision>
+      <!--<xacro:cylinder_inertial radius="0.6" length="0.12" mass="${wrist_3_mass}">
+        <origin xyz="0.0 0.0 0.0" rpy="0 0 0" />
+      </xacro:cylinder_inertial>-->
+    </link>
     <xacro:ur_arm_transmission prefix="${prefix}" />
     <xacro:ur_arm_gazebo prefix="${prefix}" />
