Commit message: EEF-URDF-File added. Files sorted, renamed and moved to .old

File: coffee_on_table/urdf/butler_robot.urdf.xacro (robot description, xacro)
@@ -10,5 +10,5 @@
   <!-- ur5 -->
   <xacro:include filename="$(find ur_description)/urdf/ur5.urdf.xacro" />
-  <!--NOT LIMITED<xacro:ur5_robot prefix="" joint_limited="false"/>-->
+  <!-- UNCOMMENT FOR NOT LIMITED <xacro:ur5_robot prefix="" joint_limited="false"/>-->
   <xacro:ur5_robot prefix="" joint_limited="true"
     shoulder_pan_lower_limit="${-pi}" shoulder_pan_upper_limit="${pi}"
@@ -21,4 +21,6 @@
   <!-- Controlbox -->
   <xacro:include filename="$(find coffee_on_table)/urdf/controlbox.urdf" />
+  <!-- EEF -->
+  <xacro:include filename="$(find coffee_on_table)/urdf/eef.urdf" />
   <!-- Connection UR to planning frame world -->
   <link name="world" />
@@ -28,7 +30,7 @@
     <origin xyz="0.0 0.0 0.0" rpy="0.0 0.0 0.0" />
   </joint>
-  <!-- Connection MiR to world where UR is connected -->
+  <!-- Connection MiR to planning frame world where UR is connected -->
   <joint name="compJoint" type="fixed">
-    <origin xyz="0.153 -0.0325 0.892" rpy="0 0 0" /> <!-- 0.153 = 0.038 + 0.115; - ; 0.892 = 0.352 + 0.54-->
+    <origin xyz="0.153 -0.0325 0.892" rpy="0 0 0" /> <!-- Caluculations: from base_footprint to surface 0.153 = 0.038 + 0.115; - ; 0.892 = 0.352 + 0.54-->
     <parent link="base_link" />
     <child link="world" />
@@ -40,3 +42,15 @@
     <child link="controlbox" />
   </joint>
+  <!-- Connection UR to EEF -->
+  <joint name="eef_fixed_joint" type="fixed">
+    <parent link="wrist_3_link" />
+    <child link="eef" />
+    <origin xyz="0.0 0.0823  0.0" rpy="${pi/2.0} 0.0 ${pi/2.0}" /> <!-- 0.0823 = wrist_3_length -->
+  </joint>
+  <!-- Connection of gripper-frame to EEF to set TCP -->
+  <joint name="gripper_fixed_joint" type="fixed">
+    <parent link="wrist_3_link" />
+    <child link= "gripper" />
+    <origin xyz="0.0 ${0.0823 + 0.144} 0.0" rpy="0.0 0.0 ${pi/2.0}" />
+  </joint>
 </robot>

File: universal_robot/ur_description/urdf/ur5.urdf.xacro (robot description, xacro)
@@ -291,42 +291,4 @@
       </collision>
     </link>
-    <!-- Added for planning with gripper as eef -->
-    <joint name="${prefix}gripper_fixed_joint" type="fixed">
-      <parent link="${prefix}wrist_3_link" />
-      <child link = "${prefix}gripper" />
-      <origin xyz="0.0 ${wrist_3_length + 0.144} 0.0" rpy="0.0 0.0 ${pi/2.0}" />
-    </joint>
-    <link name="${prefix}gripper">
-      <collision>
-        <geometry>
-          <box size="0.01 0.01 0.01"/>
-        </geometry>
-        <origin rpy="0 0 0" xyz="-0.01 0 0"/>
-      </collision>
-    </link>
-    <!-- Added for showing eef -->
-    <joint name="${prefix}eef_fixed_joint" type="fixed">
-      <parent link="${prefix}wrist_3_link" />
-      <child link = "${prefix}eef" />
-      <origin xyz="0.0 ${wrist_3_length} 0.0" rpy="${pi/2.0} 0.0 ${pi/2.0}" />
-    </joint>
-    <link name="${prefix}eef">
-      <visual>
-        <geometry>
-          <mesh filename="package://ur_description/meshes/EEF.STL" scale="0.001 0.001 0.001"/>
-        </geometry>
-        <material name="LightGrey">
-          <color rgba="0.7 0.7 0.7 1.0"/>
-        </material>
-      </visual>
-      <collision>
-        <geometry>
-          <mesh filename="package://ur_description/meshes/EEF.STL" scale="0.001 0.001 0.001"/>
-        </geometry>
-      </collision>
-      <!--<xacro:cylinder_inertial radius="0.6" length="0.12" mass="${wrist_3_mass}">
-        <origin xyz="0.0 0.0 0.0" rpy="0 0 0" />
-      </xacro:cylinder_inertial>-->
-    </link>
     <xacro:ur_arm_transmission prefix="${prefix}" />
     <xacro:ur_arm_gazebo prefix="${prefix}" />
