Commit message: Renamed Package from coffee_on_table to butler

File: butler/urdf/butler_robot.urdf.xacro (robot description, xacro)
@@ -20,7 +20,7 @@
   />
   <!-- Controlbox -->
-  <xacro:include filename="$(find coffee_on_table)/urdf/controlbox.urdf" />
+  <xacro:include filename="$(find butler)/urdf/controlbox.urdf" />
   <!-- EEF -->
-  <xacro:include filename="$(find coffee_on_table)/urdf/eef.urdf" />
+  <xacro:include filename="$(find butler)/urdf/eef.urdf" />
   <!-- Connection UR to planning frame world -->
   <link name="world" />

File: butler/urdf/eef.urdf (robot description, URDF)
Before this commit: robot eef, 2 links, 0 joints
Links:
- link eef: geometry collision mesh filename=package://butler/urdf/meshes/EEF.STL scale=0.001 0.001 0.001; visual mesh filename=package://butler/urdf/meshes/EEF.STL scale=0.001 0.001 0.001

Commit message: Changes to grab cup

File: butler/urdf/butler_robot.urdf.xacro (robot description, xacro)
@@ -33,4 +33,5 @@
   <joint name="compJoint" type="fixed">
     <origin xyz="0.153 -0.0325 0.892" rpy="0 0 0" /> <!-- Caluculations: from base_footprint to surface 0.153 = 0.038 + 0.115; - ; 0.892 = 0.352 + 0.54-->
+    <!--<origin xyz="0.093 -0.0125 0.892" rpy="0 0 0" />-->
     <parent link="base_link" />
     <child link="world" />
